Commit message: Cleaned up the code a little and added comments

File: src/terrapin/terrapin_description/urdf/terrapin.gazebo.xacro (robot description, xacro)
@@ -19,46 +19,4 @@
       <wheelTorque>10</wheelTorque>
     </plugin>
-  </gazebo>
-  <gazebo reference="base_link">
-    <material>Gazebo/Grey</material>
-  </gazebo>
-  <!-- Physics Data? -->
-  <gazebo reference="wheel_left_link">
-    <mu1>10</mu1>
-    <mu2>10</mu2>
-    <kp>500000.0</kp>
-    <kd>10.0</kd>
-    <minDepth>0.001</minDepth>
-    <maxVel>0.1</maxVel>
-    <fdir1>1 0 0</fdir1>
-    <material>Gazebo/DarkGrey</material>
-  </gazebo>
-  <gazebo reference="wheel_right_link">
-    <mu1>10</mu1>
-    <mu2>10</mu2>
-    <kp>500000.0</kp>
-    <kd>10.0</kd>
-    <minDepth>0.001</minDepth>
-    <maxVel>0.1</maxVel>
-    <fdir1>1 0 0</fdir1>
-    <material>Gazebo/DarkGrey</material>
-  </gazebo>
-  <gazebo reference="caster_back_right_link">
-    <mu1>0.0</mu1>
-    <mu2>0.0</mu2>
-    <kp>1000000.0</kp>
-    <kd>100.0</kd>
-    <minDepth>0.001</minDepth>
-    <maxVel>1.0</maxVel>
-    <material>Gazebo/Grey</material>
-  </gazebo>
-  <gazebo reference="caster_back_left_link">
-    <mu1>0.0</mu1>
-    <mu2>0.0</mu2>
-    <kp>1000000.0</kp>
-    <kd>100.0</kd>
-    <minDepth>0.001</minDepth>
-    <maxVel>1.0</maxVel>
-    <material>Gazebo/Grey</material>
   </gazebo>
   <!-- IMU -->
@@ -97,37 +55,4 @@
     </sensor>
     <material>Gazebo/Grey</material>
-  </gazebo>
-  <!-- LDS LFCD Sensor -->
-  <gazebo reference="base_scan">
-    <material>Gazebo/DarkGrey</material>
-    <sensor type="ray" name="lds_lfcd_sensor">
-      <pose>0 0 0 0 0 0</pose>
-      <visualize>$(arg laser_visual)</visualize>
-      <update_rate>1800</update_rate>
-      <ray>
-        <scan>
-          <horizontal>
-            <samples>360</samples>
-            <resolution>1</resolution>
-            <min_angle>0.0</min_angle>
-            <max_angle>6.28</max_angle>
-          </horizontal>
-        </scan>
-        <range>
-          <min>0.120</min>
-          <max>3.5</max>
-          <resolution>0.015</resolution>
-        </range>
-        <noise>
-          <type>gaussian</type>
-          <mean>0.0</mean>
-          <stddev>0.01</stddev>
-        </noise>
-      </ray>
-      <plugin name="gazebo_ros_lds_lfcd_controller" filename="libgazebo_ros_laser.so">
-        <topicName>/scan</topicName>
-        <frameName>base_scan</frameName>
-      </plugin>
-    </sensor>
   </gazebo>
   <!-- Realsense R200 -->
@@ -175,3 +100,75 @@
     </sensor>
   </gazebo>
+  <!-- LDS LFCD Sensor -->
+  <gazebo reference="base_scan">
+    <material>Gazebo/DarkGrey</material>
+    <sensor type="ray" name="lds_lfcd_sensor">
+      <pose>0 0 0 0 0 0</pose>
+      <visualize>$(arg laser_visual)</visualize>
+      <update_rate>1800</update_rate>
+      <ray>
+        <scan>
+          <horizontal>
+            <samples>360</samples>
+            <resolution>1</resolution>
+            <min_angle>0.0</min_angle>
+            <max_angle>6.28</max_angle>
+          </horizontal>
+        </scan>
+        <range>
+          <min>0.120</min>
+          <max>3.5</max>
+          <resolution>0.015</resolution>
+        </range>
+        <noise>
+          <type>gaussian</type>
+          <mean>0.0</mean>
+          <stddev>0.01</stddev>
+        </noise>
+      </ray>
+      <plugin name="gazebo_ros_lds_lfcd_controller" filename="libgazebo_ros_laser.so">
+        <topicName>/scan</topicName>
+        <frameName>base_scan</frameName>
+      </plugin>
+    </sensor>
+  </gazebo>
+  <!-- Physics Data -->
+  <gazebo reference="wheel_left_link">
+    <mu1>10</mu1>
+    <mu2>10</mu2>
+    <kp>500000.0</kp>
+    <kd>10.0</kd>
+    <minDepth>0.001</minDepth>
+    <maxVel>0.1</maxVel>
+    <fdir1>1 0 0</fdir1>
+    <material>Gazebo/DarkGrey</material>
+  </gazebo>
+  <gazebo reference="wheel_right_link">
+    <mu1>10</mu1>
+    <mu2>10</mu2>
+    <kp>500000.0</kp>
+    <kd>10.0</kd>
+    <minDepth>0.001</minDepth>
+    <maxVel>0.1</maxVel>
+    <fdir1>1 0 0</fdir1>
+    <material>Gazebo/DarkGrey</material>
+  </gazebo>
+  <gazebo reference="caster_back_right_link">
+    <mu1>0.0</mu1>
+    <mu2>0.0</mu2>
+    <kp>1000000.0</kp>
+    <kd>100.0</kd>
+    <minDepth>0.001</minDepth>
+    <maxVel>1.0</maxVel>
+    <material>Gazebo/Grey</material>
+  </gazebo>
+  <gazebo reference="caster_back_left_link">
+    <mu1>0.0</mu1>
+    <mu2>0.0</mu2>
+    <kp>1000000.0</kp>
+    <kd>100.0</kd>
+    <minDepth>0.001</minDepth>
+    <maxVel>1.0</maxVel>
+    <material>Gazebo/Grey</material>
+  </gazebo>
 </robot>

File: src/terrapin/terrapin_description/urdf/terrapin.main.xacro (robot description, xacro)
@@ -12,5 +12,7 @@
     <origin xyz="0 0 0.010" rpy="0 0 0"/>
   </joint>
+  <!-- Base Link -->
   <link name="base_link">
+    <xacro:gz_grey_material name="base_link"/>
     <visual>
       <origin xyz="-0.064 0 0.0" rpy="0 0 0"/>
@@ -34,4 +36,5 @@
     </inertial>
   </link>
+  <!-- Wheels -->
   <joint name="wheel_left_joint" type="continuous">
     <parent link="base_link"/>
@@ -90,4 +93,5 @@
     </inertial>
   </link>
+  <!-- Casters -->
   <joint name="caster_back_right_joint" type="fixed">
     <parent link="base_link"/>
@@ -130,4 +134,5 @@
     </inertial>
   </link>
+  <!-- IMU -->
   <joint name="imu_joint" type="fixed">
     <parent link="base_link"/>
@@ -141,4 +146,5 @@
     <origin xyz="-0.064 0 0.121" rpy="0 0 0"/>
   </joint>
+  <!-- Base Scan -->
   <link name="base_scan">
     <visual>
@@ -163,4 +169,5 @@
     </inertial>
   </link>
+  <!-- Camera -->
   <joint name="camera_joint" type="fixed">
     <origin xyz="0.064 -0.065 0.094" rpy="0 0 0"/>

File: src/terrapin/terrapin_description/urdf/terrapin.materials.xacro (robot description, xacro)
@@ -31,3 +31,29 @@
     <color rgba="1.0 1.0 1.0 1.0"/>
   </material>
+  <!-- Gazebo Materials -->
+  <xacro:macro name="gz_black_material" params="name">
+    <gazebo reference="${name}">
+      <material>Gazebo/FlatBlack</material>
+    </gazebo>
+  </xacro:macro>
+  <xacro:macro name="gz_grey_material" params="name">
+    <gazebo reference="${name}">
+      <material>Gazebo/Grey</material>
+    </gazebo>
+  </xacro:macro>
+  <xacro:macro name="gz_white_material" params="name">
+    <gazebo reference="${name}">
+      <material>Gazebo/White</material>
+    </gazebo>
+  </xacro:macro>
+  <xacro:macro name="gz_blue_material" params="name">
+    <gazebo reference="${name}">
+      <material>Gazebo/Blue</material>
+    </gazebo>
+  </xacro:macro>
+  <xacro:macro name="gz_red_material" params="name">
+    <gazebo reference="${name}">
+      <material>Gazebo/Red</material>
+    </gazebo>
+  </xacro:macro>
 </robot>
